File: Hardware/Tp_kicad/Tp_kicad.kicad_pcb (KiCad board)
At the start: 2 copper layers, 58 x 48 mm, 27 parts, among them J1 Conn_02x07_Odd_Even, J2 Conn_01x02, J3 Conn_01x02, J4 Conn_01x02, U1 STM32L021K4Tx, U2 BU33SD5WG-TR, U3 MCP4801

Commit message: commmit
Parts:
- moved C1 34.2 mm to (117.8, 103.4), turned to -90 degrees
- moved R1 22.6 mm to (128.3, 83.1)
- moved C5 22.3 mm to (120.9, 91.7)
- moved C3 20.6 mm to (144.5, 93.5), turned to -90 degrees
- moved C7 18.0 mm to (122.4, 73.2), turned to 0 degrees
- moved C2 17.4 mm to (129.2, 86.3), turned to 90 degrees
- moved R2 14.5 mm to (146.1, 86.1), turned to 180 degrees
- moved C9 13.4 mm to (149.4, 106.0), turned to -90 degrees
- moved C10 11.8 mm to (147.4, 106.0), turned to -90 degrees
- moved C4 11.7 mm to (126.2, 91.7)
- moved L1 11.4 mm to (122.7, 102.4), turned to 0 degrees
- moved U3 10.9 mm to (146.8, 101.3), turned to 180 degrees
- moved D2 10.2 mm to (122.2, 76.5), turned to 180 degrees
- moved D1 8.01 mm to (146.3, 84.3), turned to 180 degrees
- moved R3 6.43 mm to (122.2, 78.7), turned to 180 degrees
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Routing:
- net +3.3V: track 43.3 -> 145.0 mm, vias 0 -> 2
- net +3.3VA: track 0.00 -> 62.0 mm, vias 0 -> 2
- net /USART2_RX: track 0.00 -> 58.1 mm
- net /ADC_IN1: track 0.00 -> 49.6 mm
- net /NRST: track 5.80 -> 41.4 mm
- net /USART2_TX: track 0.00 -> 26.4 mm, vias 0 -> 2
- net /DAC_OUT: track 0.00 -> 25.4 mm, vias 0 -> 1
- net Net-(D1-K): track 25.1 -> 1.83 mm
- net /DAC_nCS: track 0.91 -> 21.2 mm
- net /SPI1_SCK: track 0.00 -> 19.2 mm
- net /SWDIO: track 0.00 -> 17.1 mm
- net /SPI1_MOSI: track 0.00 -> 17.0 mm
- net /SWDCLK: track 0.00 -> 15.2 mm
- net /DAC_nLDAC: track 0.00 -> 14.9 mm
- net +5V: track 58.0 -> 44.6 mm
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Other:
- board text added: "TT.BP"
